File: mc34063-step-down-dev-0.1-RELEASED/mc34063-step-down-dev-0.1.kicad_sch (KiCad schematic)
At the start: 14 parts, among them J1 M, J2 M, J3 M, J4 M, U1 MC34063AD, U2 220uH

Commit message: released dev board
Parts:
- removed J1, J2, J3, J4: M, Connector_Pin:Pin_D1.2mm_L10.2mm_W2.9mm_FlatFork, symbol Connector_Generic:Conn_01x01
- added J1, J2, J3, J4: Conn_01x02, TerminalBlock:TerminalBlock_bornier-2_P5.08mm, symbol Connector_Generic:Conn_01x02
- added TP1, TP2, TP3: TestPoint, TestPoint:TestPoint, symbol Connector:TestPoint
Connections:
- net GND: now also J1.1 (Pin_1), J4.2 (Pin_2)
- net In: now also J1.2 (Pin_2), J2.1 (Pin_1); no longer Ci1.1, RSC1.1, U1.6 (Vin)
- net Vfeedback: now also TP3.1
- net Vout: now also J3.2 (Pin_2), J4.1 (Pin_1); no longer Co1.1, Co2.1, R1.1, U2.2
- net at Ct1.1, U1.3 (TC): now also TP1.1
- net at D1.1 (K), U1.2 (SwE), U2.1: now also TP2.1
- new net: Co1.1, Co2.1, J3.1 (Pin_1), R1.1, U2.2
- new net: Ci1.1, J2.2 (Pin_2), RSC1.1, U1.6 (Vin)
