File: mc34063-step-down-dev-0.2/mc34063-step-down-dev-0.2.kicad_sch (KiCad schematic)
At the start: 14 parts, among them J1 M, J2 M, J3 M, J4 M, U1 MC34063AD, U2 220uH

Commit message: updates
Parts:
- removed J1, J2, J3, J4: M, Connector_Pin:Pin_D1.2mm_L10.2mm_W2.9mm_FlatFork, symbol Connector_Generic:Conn_01x01
- removed U2: 220uH, mc34063-power-inductor:mc34063-power-inductor, symbol mc34063-power-inductor:mc34063-power-inductor
- added Co2: 470u/10V, Capacitor_SMD:CP_Elec_6.3x7.7, symbol Device:C_Polarized
- added Co3, Co5: 47u/10V, Capacitor_SMD:C_1206_3216Metric_Pad1.33x1.80mm_HandSolder, symbol Device:C
- added U2: mc34063-power-inductor-leaded, mc34063-power-inductor-leaded:mc34063-power-inductor-leaded, symbol mc34063-power-inductor-leaded:mc34063-power-inductor-leaded
- added U3, U4, U5, U6: 1pin, 1pin:1pin, symbol 1pin:1pin
- renumbered Co2 to Co4
Connections:
- net GND: now also Co2.2, Co3.2, Co5.2, U4.1, U6.1
- net at D1.1 (K), U1.2 (SwE): now also U2.2
- net In: no longer names the net of Ci1.1, RSC1.1, U1.6 (Vin)
- net In: now also U3.1
- net Vout: no longer names the net of Co1.1, Co4.1, R1.1
- net Vout: now also Co2.1, Co3.1, Co5.1, U2.1, U5.1
Other:
- moved on the sheet: Co4
